File: LoRa-GW-FeatherWing.kicad_sch (KiCad schematic)
At the start: 116 parts, among them J1 Conn_Coaxial, J2 Conn_Coaxial, U1 SX1303IMLTRT, U2 SX1250, U3 SX1250, U4 TPS7A91, U5 JT255BI0032.000000, U6 TLV62568DRL, U7 SKY66420-11, U8 EVA-8M

Commit message: Adding SX1261 for LBT
Parts:
- added C36: 3pF, Capacitor_SMD:C_0201_0603Metric, symbol Device:C
- added C66, C67: 3.6pF, Capacitor_SMD:C_0201_0603Metric, symbol Device:C
- added C68: 10pF, Capacitor_SMD:C_0201_0603Metric, symbol Device:C
- added C69, C70: 1uF, Capacitor_SMD:C_0402_1005Metric, symbol Device:C
- added C71: 470nF, Capacitor_SMD:C_0402_1005Metric, symbol Device:C
- added D5, D6: D_TVS, Diode_SMD:D_0402_1005Metric, symbol Device:D_TVS
- added L18: 18nH, Inductor_SMD:L_0201_0603Metric, symbol Device:L
- added L19: MLZ2012N150LT000, Inductor_SMD:L_0805_2012Metric, symbol Device:L
- added L20: FB, Inductor_SMD:L_0201_0603Metric, symbol Device:L
- added R18, R19: 100K, Resistor_SMD:R_0201_0603Metric, symbol Device:R
- added R20, R21, R22, R23, R24: 220R, Resistor_SMD:R_0201_0603Metric, symbol Device:R
- added U10: TMP117AIYBGR, SX1302:TMP117AIYBGR, symbol 2021-03-06_06-12-35:TMP117AIYBGR
- added U9: SX1262IMLTRT, SX1302:SX1262IMLTRT, symbol 2021-03-08_06-26-18:SX1262IMLTRT
- C33, C35: footprint Capacitor_SMD:C_0402_1005Metric -> Capacitor_SMD:C_0603_1608Metric
- C60: value 0R -> DNP
- C61: footprint Capacitor_SMD:C_0201_0603Metric -> Capacitor_SMD:C_0402_1005Metric
- L16: footprint Inductor_SMD:L_0201_0603Metric -> Inductor_SMD:L_0402_1005Metric
Connections:
- net +3V3: now also C2.1, C4.1, U2.10 (VBAT_DIO), U2.9 (VBAT_RF), U3.10 (VBAT_DIO), U3.9 (VBAT_RF), L20.2; no longer C62.1, U5.4 (VDD)
- net GND: now also C60.2, C36.1, C67.1, C69.2, C70.2, C71.2, D5.1 (A1), D6.1 (A1), R22.1, U10.4 (GND), U10.5 (ADD0), U9.2 (GND), U9.20 (GND), U9.25 (GND), U9.5 (GND), U9.8 (GND); no longer U5.1 (Standby)
- net HOST_MISO: now also U9.16 (MISO)
- net HOST_MOSI: now also U9.17 (MOSI)
- net HOST_SCK: now also U9.18 (SCK)
- net TCXO_32Mhz: now also R20.2
- net VDD_RF: now also C36.2, C69.1, C70.1, R18.2, R19.2, R23.1, R24.1, U10.3 (V+), U9.1 (VDD_IN), U9.10 (VBAT), U9.11 (VBAT_IO); no longer C2.1, C4.1, U2.10 (VBAT_DIO), U2.9 (VBAT_RF), U3.10 (VBAT_DIO), U3.9 (VBAT_RF)
- net SX1261_DIO1: now reaches U1.54 (GPIO7)
- net SX1261_DIO1: now also A1.7 (A2), U9.13 (DIO1)
- net at U1.58 (GPIO5): no longer R11.2
- net at U1.59 (GPIO4): now also R11.2; no longer R12.2
- net at U1.60 (GPIO3): no longer R13.2
- net at U1.63 (GPIO2): now also R12.2
- net at U1.66 (GPIO0): now also R13.2
- net at J2.1 (In), L16.2: now also U8.1 (ANT), D6.2 (A2); no longer C60.1
- net at C45.2, J1.1 (In), L13.2: now also D5.2 (A2)
- net at C15.1, C16.1, C18.1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: now also C60.1, C66.1
- net SDA: now reaches A1.17 (SDA)
- net SDA: now also R19.1, U10.1 (SDA)
- net SCL: now reaches A1.18 (SCL)
- net SCL: now also R18.1, U10.2 (SCL)
- net SX1262_RESET: now reaches A1.6 (A1)
- net SX1262_RESET: now also R23.2, U9.15 (NRESET)
- net SX1261_BUSY: now reaches A1.8 (A3)
- net SX1261_BUSY: now also U9.14 (BUSY)
- net SX1261_CSN: now reaches A1.9 (A4)
- net SX1261_CSN: now also R24.2, U9.19 (NSS)
- new net: C62.1, L20.1, R21.2, U5.4 (VDD)
- new net: L19.1, U9.9 (DCC_SW)
- new net: C71.1, L19.2, U9.7 (VREG)
- new net: C67.2, L18.1, U9.22 (RFI_N)
- new net: C66.2, L18.2, U9.21 (RFI_P)
- new net: C68.1, U9.3 (XTA)
- new net: C68.2, R20.1
- new net: R21.1, R22.2, U5.1 (Standby)
Other:
- note added: "Temperature Sensor"
- moved on the sheet: C1, C10, C11, C12, C13, C14, C15, C16, C17, C18, C19, C2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
